File: pcb/riser/riser.kicad_pcb (KiCad board)
At the start: 2 copper layers, 100 x 90 mm, 29 parts, among them CN1 Molex_52602_0579, CN2 CONN_02X20, CN3 CONN_02X20, CN4 CONN_02X22, CN5 CONN_01X09, CN6 USB-A, P1 CONN_01X02, P2 CONN_01X02, P3 CONN_01X02, X1 11.2896M

Commit message: Tweak mounting hole positions
Parts:
- moved REF** 0.12 mm to (199.2, 48.7)
- moved REF** 0.11 mm to (131.0, 48.7)
- moved REF** 0.09 mm to (199.2, 116.9)
- moved REF** 0.06 mm to (131.0, 116.9)
Other:
- board text added: "v2.1"
- board text removed: "v2.0"
Changed lines of the file:
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@@
     (links 147)
     (no_connects 0)
-    (area 125.924999 43.924999 226.075001 134.075001)
+    (area 121.377857 32.65 242.5 134.229)
     (thickness 1.6)
     (drawings 52)
@@
   )
   (module Mounting_Holes:MountingHole_3.2mm_M3 (layer F.Cu)
-    (at 199.136 48.833)
+    (at 199.21 48.734)
     (descr "Mounting Hole 3.2mm, no annular, M3")
     (tags "mounting hole 3.2mm no annular m3")
@@
   )
   (module Mounting_Holes:MountingHole_3.2mm_M3 (layer F.Cu)
-    (at 131.064 48.833)
+    (at 131.02 48.734)
     (descr "Mounting Hole 3.2mm, no annular, M3")
     (tags "mounting hole 3.2mm no annular m3")
@@
   )
   (module Mounting_Holes:MountingHole_3.2mm_M3 (layer F.Cu)
-    (at 131.064 116.967)
+    (at 131.02 116.924)
     (descr "Mounting Hole 3.2mm, no annular, M3")
     (tags "mounting hole 3.2mm no annular m3")
@@
   )
   (module Mounting_Holes:MountingHole_3.2mm_M3 (layer F.Cu)
-    (at 199.136 116.967)
+    (at 199.21 116.924)
     (descr "Mounting Hole 3.2mm, no annular, M3")
     (tags "mounting hole 3.2mm no annular m3")
@@
     (effects (font (size 1.5 1.5) (thickness 0.3)))
   )
-  (gr_text v2.0 (at 130.2 131.2) (layer F.SilkS)
+  (gr_text v2.1 (at 130.2 131.2) (layer F.SilkS)
     (effects (font (size 1.5 1.5) (thickness 0.3)))
   )

Commit message: Decrease via drill size to get a larger annular ring
Routing:
- net GND: vias 1 -> 0
Other:
- net class Default: via_drill 0.635 -> 0.381
- net class LED: via_drill 0.635 -> 0.381
- net class Power: via_drill 0.635 -> 0.381

Commit message: Updating the schematic file to include the new style of referencing kicad components with some minor aesthetic changes. Also updating orientation of the LED in the PCB.
Parts:
- moved D1 2.60 mm to (214.5, 130.2), turned to 0 degrees
Connections:
- D1 pad 1: Net-(D1-Pad1) -> /ACTIVEn
- D1 pad 2: /ACTIVEn -> Net-(D1-Pad2)
- R8 pad 2: Net-(D1-Pad1) -> Net-(D1-Pad2)
Routing:
- net Net-(D1-Pad2): track 0.00 -> 3.82 mm
- net Net-(D1-Pad1): track 3.82 -> 0.00 mm

Commit message: v2.2
Other:
- board text added: "v2.2"
- board text removed: "v2.1"
Changed lines of the file:
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@@
-(kicad_pcb (version 20171130) (host pcbnew 5.1.2)
+(kicad_pcb (version 20171130) (host pcbnew 5.1.5)
   (general
     (thickness 1.6)
@@
     (visible_elements FFFFFF7F)
     (pcbplotparams
-      (layerselection 0x010f0_80000001)
+      (layerselection 0x010f0_ffffffff)
       (usegerberextensions false)
       (usegerberattributes false)
@@
     (effects (font (size 1.5 1.5) (thickness 0.3)))
   )
-  (gr_text v2.1 (at 130.2 131.2) (layer F.SilkS)
+  (gr_text v2.2 (at 130.2 131.2) (layer F.SilkS)
     (effects (font (size 1.5 1.5) (thickness 0.3)))
   )
@@
   (segment (start 208.25 114.15) (end 207 115.4) (width 0.4) (layer F.Cu) (net 73))
   (segment (start 214.52 130.34) (end 214.56 130.3) (width 0.4) (layer F.Cu) (net 73))
-  (segment (start 217.1 130.3) (end 220.84 130.3) (width 0.4) (layer F.Cu) (net 84))
-  (segment (start 220.84 130.3) (end 220.9 130.36) (width 0.2032) (layer F.Cu) (net 84))
   (segment (start 190 124.82) (end 192.22 124.82) (width 0.6) (layer F.Cu) (net 78))
   (segment (start 202.65 131.55) (end 202.65 130.05) (width 0.6) (layer F.Cu) (net 78))
@@
   (segment (start 180.75 129.55) (end 179.5 130.8) (width 0.6) (layer F.Cu) (net 82))
   (segment (start 180.89 127.54) (end 180.75 127.4) (width 0.2032) (layer F.Cu) (net 82))
+  (segment (start 217.1 130.3) (end 220.84 130.3) (width 0.4) (layer F.Cu) (net 84))
+  (segment (start 220.84 130.3) (end 220.9 130.36) (width 0.2032) (layer F.Cu) (net 84))
 )
